Commit message: modify weight

File: urdf/andbot.xacro (robot description, xacro)
@@ -33,5 +33,5 @@
     <inertial>
       <origin xyz="0 0 0.00" rpy="0 0 0"/>
-      <mass value="1"/>
+      <mass value="1.5"/>
       <inertia ixx="0.248" ixy="0" ixz="0" iyy="0.248" iyz="0" izz="0.748"/>
     </inertial>
@@ -78,5 +78,5 @@
     <inertial>
       <origin xyz="0 0 0.00" rpy="0 0 0"/>
-      <mass value="10"/>
+      <mass value="3.5"/>
       <inertia ixx="0.248" ixy="0" ixz="0" iyy="0.248" iyz="0" izz="0.748"/>
     </inertial>
@@ -110,5 +110,5 @@
     <inertial>
       <origin xyz="0 0 0.00" rpy="0 0 0"/>
-      <mass value="1"/>
+      <mass value="0.75"/>
       <inertia ixx="0.148" ixy="0" ixz="0" iyy="0.148" iyz="0" izz="0.748"/>
     </inertial>
@@ -142,5 +142,5 @@
     <inertial>
       <origin xyz="0 0 0.00" rpy="0 0 0"/>
-      <mass value="1"/>
+      <mass value="0.75"/>
       <inertia ixx="0.148" ixy="0" ixz="0" iyy="0.148" iyz="0" izz="0.748"/>
     </inertial>
@@ -174,5 +174,5 @@
     <inertial>
       <origin xyz="0 0 0.00" rpy="0 0 0"/>
-      <mass value="1"/>
+      <mass value="0.75"/>
       <inertia ixx="0.148" ixy="0" ixz="0" iyy="0.148" iyz="0" izz="0.748"/>
     </inertial>
@@ -206,5 +206,5 @@
     <inertial>
       <origin xyz="0 0 0.00" rpy="0 0 0"/>
-      <mass value="1"/>
+      <mass value="0.75"/>
       <inertia ixx="0.148" ixy="0" ixz="0" iyy="0.148" iyz="0" izz="0.748"/>
     </inertial>
@@ -238,5 +238,5 @@
     <inertial>
       <origin xyz="0 0 0.07" rpy="0 0 0"/>
-      <mass value="10"/>
+      <mass value="12"/>
       <inertia ixx="0.248" ixy="0" ixz="0" iyy="0.748" iyz="0" izz="0.748"/>
     </inertial>
@@ -264,5 +264,5 @@
     <inertial>
       <origin xyz="0 0 0" rpy="0 0 0"/>
-      <mass value="0.5"/>
+      <mass value="0.05"/>
       <inertia ixx="0.0098" ixy="0" ixz="0" iyy="0.0098" iyz="0" izz="0.0098"/>
     </inertial>
@@ -300,5 +300,5 @@
     </visual>
     <inertial>
-      <mass value="0.1"/>
+      <mass value="0.002"/>
       <origin xyz="0 0 0" rpy="0 0 0"/>
       <inertia ixx="1e-6" ixy="0" ixz="0" iyy="1e-6" iyz="0" izz="0.01"/>
@@ -330,5 +330,5 @@
     <inertial>
       <origin xyz="0 0 0" rpy="0 1.570795 1.570795"/>
-      <mass value="0.2"/>
+      <mass value="0.4"/>
       <inertia ixx="0.0135" ixy="0" ixz="0" iyy="0.0135" iyz="0" izz="0.025"/>
     </inertial>
@@ -381,5 +381,5 @@
     <inertial>
       <origin xyz="0 0 0" rpy="0 1.570795 1.570795"/>
-      <mass value="0.2"/>
+      <mass value="0.4"/>
       <inertia ixx="0.0135" ixy="0" ixz="0" iyy="0.0135" iyz="0" izz="0.025"/>
     </inertial>
@@ -881,9 +881,9 @@
         <scan>
           <horizontal>
-            <samples>750</samples>
+            <samples>720</samples>
             <resolution>1</resolution>
-            <min_angle>${-PI/2}</min_angle>
+            <min_angle>-1</min_angle>
             <!-- -0.0174532925 -->
-            <max_angle>${PI/2}</max_angle>
+            <max_angle>1</max_angle>
             <!-- 0.0174532925 -->
           </horizontal>

Commit message: create two ir beam but no rotate

File: urdf/andbot.xacro (robot description, xacro)
@@ -1,3 +1,4 @@
 <?xml version="1.0"?>
+<!--before install IR andbot-->
 <robot xmlns:xacro="http://www.ros.org/wiki/xacro" name="andbot">
   <xacro:property name="PI" value="3.1415926535897931"/>
@@ -14,4 +15,191 @@
     <child link="base_link"/>
   </joint>
+<!-- Testing for IR obstacle avoidance-->
+<!-- Testing for IR obstacle avoidance-->
+<!-- Testing for IR obstacle avoidance-->
+<!-- Testing for IR obstacle avoidance-->
+<!-- ir_up plugin -->
+  <gazebo reference="ir_up">
+    <mu1>1.0</mu1>
+    <mu2>1.0</mu2>
+    <material>Gazebo/Yellow</material>
+    <sensor type="ray" name="head_hokuyo_sensor">
+      <pose>0 0 0 0 0 0</pose>
+      <visualize>true</visualize>
+      <update_rate>100</update_rate>
+      <ray>
+        <scan>
+          <horizontal>
+            <samples>3</samples>
+            <resolution>1</resolution>
+            <min_angle>-0.001</min_angle>
+            <!-- -0.0174532925 -->
+            <max_angle>0.001</max_angle>
+            <!-- 0.0174532925 -->
+          </horizontal>
+        </scan>
+        <range>
+          <min>0.10</min>
+          <max>3.0</max>
+          <resolution>0.01</resolution>
+        </range>
+        <noise>
+          <type>gaussian</type>
+          <!-- Noise parameters based on published spec for Hokuyo laser
+		       achieving "+-30mm" accuracy at range < 10m.  A mean of 0.0m and
+		       stddev of 0.01m will put 99.7% of samples within 0.03m of the true
+		       reading. -->
+          <mean>0.0</mean>
+          <stddev>0.00</stddev>
+        </noise>
+      </ray>
+      <plugin name="gazebo_ros_head_hokuyo_controller" filename="libgazebo_ros_laser.so">
+        <topicName>ir_up_dist</topicName>
+        <frameName>ir_up</frameName>
+      </plugin>
+    </sensor>
+  </gazebo>
+  <!-- Body link /ir Link joint -->
+  <joint name="ir_up_joint" type="continuous">
+    <parent link="body_link"/>
+    <child link="ir_up"/>
+    <origin xyz="${0.145/2} 0 ${0.875-0.029}" rpy="3.14 ${1.57/2} 0"/>
+    <axis xyz="0 0 1"/>
+          <limit upper="1.57" lower="-1.57" velocity="10" effort="7"/>
+	  <joint_properties damping="0.0" friction="0.0"/>
+  </joint>
+  <!-- Transmission for ir_up joint -->
+  <transmission name="ir_up_trans">
+    <type>transmission_interface/SimpleTransmission</type>
+    <joint name="ir_up_joint">
+      <hardwareInterface>EffortJointInterface</hardwareInterface>
+    </joint>
+    <actuator name="ir_up_Motor">
+      <hardwareInterface>EffortJointInterface</hardwareInterface>
+      <mechanicalWhiteuction>1</mechanicalWhiteuction>
+    </actuator>
+  </transmission>
+  <!-- IR_UP link -->
+  <link name="ir_up">
+    <collision>
+      <origin xyz="0 0 0" rpy="0 1.57 0"/>
+      <geometry>
+        <cylinder length="0.04" radius="0.01"/>
+      </geometry>
+    </collision>
+    <visual>
+      <origin xyz="0 0 0" rpy="0 1.57 0"/>
+      <geometry>
+        <cylinder length="0.04" radius="0.01"/>
+      </geometry>
+       <material name="Yellow">
+         <color rgba="1 1 0 1"/>
+       </material>
+    </visual>
+    <inertial>
+      <mass value="0.002"/>
+      <origin xyz="0 0 0" rpy="0 0 0"/>
+      <inertia ixx="1e-6" ixy="0" ixz="0" iyy="1e-6" iyz="0" izz="0.01"/>
+    </inertial>
+  </link>
+  <gazebo reference="ir_up">
+    <mu1 value="5.0"/>
+    <mu2 value="5.0"/>
+    <kp value="10000000.0"/>
+    <kd value="1.0"/>
+  </gazebo>
+<!-- ir_down plugin -->
+  <gazebo reference="ir_down">
+    <mu1>1.0</mu1>
+    <mu2>1.0</mu2>
+    <material>Gazebo/Yellow</material>
+    <sensor type="ray" name="head_hokuyo_sensor">
+      <pose>0 0 0 0 0 0</pose>
+      <visualize>true</visualize>
+      <update_rate>100</update_rate>
+      <ray>
+        <scan>
+          <horizontal>
+            <samples>3</samples>
+            <resolution>1</resolution>
+            <min_angle>-0.001</min_angle>
+            <!-- -0.0174532925 -->
+            <max_angle>0.001</max_angle>
+            <!-- 0.0174532925 -->
+          </horizontal>
+        </scan>
+        <range>
+          <min>0.10</min>
+          <max>3.0</max>
+          <resolution>0.01</resolution>
+        </range>
+        <noise>
+          <type>gaussian</type>
+          <!-- Noise parameters based on published spec for Hokuyo laser
+		       achieving "+-30mm" accuracy at range < 10m.  A mean of 0.0m and
+		       stddev of 0.01m will put 99.7% of samples within 0.03m of the true
+		       reading. -->
+          <mean>0.0</mean>
+          <stddev>0.00</stddev>
+        </noise>
+      </ray>
+      <plugin name="gazebo_ros_head_hokuyo_controller" filename="libgazebo_ros_laser.so">
+        <topicName>ir_down_dist</topicName>
+        <frameName>ir_down</frameName>
+      </plugin>
+    </sensor>
+  </gazebo>
+  <!-- Body link /ir Link joint -->
+  <joint name="ir_down_joint" type="continuous">
+    <parent link="body_link"/>
+    <child link="ir_down"/>
+    <origin xyz="${0.145/2} 0 ${0.275-0.029}" rpy="3.14 ${-1.57/2} 0"/>
+    <axis xyz="0 0 1"/>
+          <limit upper="1.57" lower="-1.57" velocity="10" effort="7"/>
+	  <joint_properties damping="0.0" friction="0.0"/>
+  </joint>
+  <!-- Transmission for ir_down joint -->
+  <transmission name="ir_down_trans">
+    <type>transmission_interface/SimpleTransmission</type>
+    <joint name="ir_down_joint">
+      <hardwareInterface>EffortJointInterface</hardwareInterface>
+    </joint>
+    <actuator name="ir_down_Motor">
+      <hardwareInterface>EffortJointInterface</hardwareInterface>
+      <mechanicalWhiteuction>1</mechanicalWhiteuction>
+    </actuator>
+  </transmission>
+  <!-- ir_down link -->
+  <link name="ir_down">
+    <collision>
+      <origin xyz="0 0 0" rpy="0 1.57 0"/>
+      <geometry>
+        <cylinder length="0.04" radius="0.01"/>
+      </geometry>
+    </collision>
+    <visual>
+      <origin xyz="0 0 0" rpy="0 1.57 0"/>
+      <geometry>
+        <cylinder length="0.04" radius="0.01"/>
+      </geometry>
+       <material name="Yellow">
+         <color rgba="1 1 0 1"/>
+       </material>
+    </visual>
+    <inertial>
+      <mass value="0.002"/>
+      <origin xyz="0 0 0" rpy="0 0 0"/>
+      <inertia ixx="1e-6" ixy="0" ixz="0" iyy="1e-6" iyz="0" izz="0.01"/>
+    </inertial>
+  </link>
+  <gazebo reference="ir_down">
+    <mu1 value="5.0"/>
+    <mu2 value="5.0"/>
+    <kp value="10000000.0"/>
+    <kd value="1.0"/>
+  </gazebo>
+<!-- End of Testing for IR obstacle avoidance-->
+<!-- End of Testing for IR obstacle avoidance-->
+<!-- End of Testing for IR obstacle avoidance-->
   <!-- Head link -->
   <link name="head_link">
@@ -40,14 +228,14 @@
     <material>Gazebo/White</material>
   </gazebo>
-  <!-- Base link /Head Link joint -->
+  <!-- Body link /Head Link joint -->
   <joint name="head_joint" type="continuous">
-    <parent link="base_link"/>
+    <parent link="body_link"/>
     <child link="head_link"/>
-    <origin xyz="-0.145 0 1.075" rpy="0 0 0"/>
+    <origin xyz="-0.145 0 ${1.075-0.029}" rpy="0 0 0"/>
     <axis xyz="0 0 1"/>
           <limit upper="1.57" lower="-1.57" velocity="10" effort="7"/>
 	  <joint_properties damping="0.0" friction="0.0"/>
   </joint>
-  <!-- Transmission for laser joint -->
+  <!-- Transmission for head joint -->
   <transmission name="head_trans">
     <type>transmission_interface/SimpleTransmission</type>

Commit message: rotate ir_ip using pos_control between -pi to pi use tow closed loop

File: urdf/andbot.xacro (robot description, xacro)
@@ -1,4 +1,3 @@
 <?xml version="1.0"?>
-<!--before install IR andbot-->
 <robot xmlns:xacro="http://www.ros.org/wiki/xacro" name="andbot">
   <xacro:property name="PI" value="3.1415926535897931"/>
@@ -64,8 +63,8 @@
     <parent link="body_link"/>
     <child link="ir_up"/>
-    <origin xyz="${0.145/2} 0 ${0.875-0.029}" rpy="3.14 ${1.57/2} 0"/>
+    <origin xyz="${0.145/2} 0 ${0.875-0.029}" rpy="0 ${0/2} 0"/>
     <axis xyz="0 0 1"/>
-          <limit upper="1.57" lower="-1.57" velocity="10" effort="7"/>
-	  <joint_properties damping="0.0" friction="0.0"/>
+          <limit upper="1.57" lower="-1.57" velocity="50" effort="2"/>
+	  <joint_properties damping="0.0" friction="0"/>
   </joint>
   <!-- Transmission for ir_up joint -->
@@ -98,7 +97,7 @@
     </visual>
     <inertial>
-      <mass value="0.002"/>
-      <origin xyz="0 0 0" rpy="0 0 0"/>
-      <inertia ixx="1e-6" ixy="0" ixz="0" iyy="1e-6" iyz="0" izz="0.01"/>
+      <mass value="0.2"/>
+      <origin xyz="0 0 0" rpy="0 0 0"/>
+      <inertia ixx="1e-6" ixy="0" ixz="0" iyy="1e-6" iyz="0" izz="0.1"/>
     </inertial>
   </link>

Commit message: ir_up can detect object in front of robot and plot in rviz using PointCloud msg

File: urdf/andbot.xacro (robot description, xacro)
@@ -39,6 +39,6 @@
         </scan>
         <range>
-          <min>0.10</min>
-          <max>3.0</max>
+          <min>0.20</min>
+          <max>1.5</max>
           <resolution>0.01</resolution>
         </range>
@@ -65,5 +65,5 @@
     <origin xyz="${0.145/2} 0 ${0.875-0.029}" rpy="0 ${0/2} 0"/>
     <axis xyz="0 0 1"/>
-          <limit upper="1.57" lower="-1.57" velocity="50" effort="2"/>
+          <limit upper="1.57" lower="-1.57" velocity="50" effort="20"/>
 	  <joint_properties damping="0.0" friction="0"/>
   </joint>
@@ -99,5 +99,5 @@
       <mass value="0.2"/>
       <origin xyz="0 0 0" rpy="0 0 0"/>
-      <inertia ixx="1e-6" ixy="0" ixz="0" iyy="1e-6" iyz="0" izz="0.1"/>
+      <inertia ixx="1e-6" ixy="0" ixz="0" iyy="1e-6" iyz="0" izz="0.005"/>
     </inertial>
   </link>
@@ -129,6 +129,6 @@
         </scan>
         <range>
-          <min>0.10</min>
-          <max>3.0</max>
+          <min>0.20</min>
+          <max>1.50</max>
           <resolution>0.01</resolution>
         </range>
@@ -155,5 +155,5 @@
     <origin xyz="${0.145/2} 0 ${0.275-0.029}" rpy="3.14 ${-1.57/2} 0"/>
     <axis xyz="0 0 1"/>
-          <limit upper="1.57" lower="-1.57" velocity="10" effort="7"/>
+          <limit upper="1.57" lower="-1.57" velocity="50" effort="2"/>
 	  <joint_properties damping="0.0" friction="0.0"/>
   </joint>
@@ -187,7 +187,7 @@
     </visual>
     <inertial>
-      <mass value="0.002"/>
-      <origin xyz="0 0 0" rpy="0 0 0"/>
-      <inertia ixx="1e-6" ixy="0" ixz="0" iyy="1e-6" iyz="0" izz="0.01"/>
+      <mass value="0.2"/>
+      <origin xyz="0 0 0" rpy="0 0 0"/>
+      <inertia ixx="1e-6" ixy="0" ixz="0" iyy="1e-6" iyz="0" izz="0.005"/>
     </inertial>
   </link>

Commit message: ir_up and ir_down sync detect object ahead of andbot

File: urdf/andbot.xacro (robot description, xacro)
@@ -6,4 +6,5 @@
   <xacro:property name="distance_between_wheels" value="0.3996"/>
   <xacro:property name="height_wheels_from_base" value="0.0392"/>
+  <xacro:property name="ir_up_angle" value="0.78539"/> <!--PI /4 -->
  <arg name="gui" value="true"/>
   <!-- Base footprint link-->
@@ -63,5 +64,5 @@
     <parent link="body_link"/>
     <child link="ir_up"/>
-    <origin xyz="${0.145/2} 0 ${0.875-0.029}" rpy="0 ${0/2} 0"/>
+    <origin xyz="${0.145/2} 0 ${0.875-0.029}" rpy="0 ${ir_up_angle} 0"/>
     <axis xyz="0 0 1"/>
           <limit upper="1.57" lower="-1.57" velocity="50" effort="20"/>
@@ -103,4 +104,39 @@
   </link>
   <gazebo reference="ir_up">
+    <mu1 value="5.0"/>
+    <mu2 value="5.0"/>
+    <kp value="10000000.0"/>
+    <kd value="1.0"/>
+  </gazebo>
+  <!-- Body link /ir up view joint -->
+  <joint name="ir_up_view_joint" type="fixed">
+    <parent link="body_link"/>
+    <child link="ir_up_view"/>
+    <origin xyz="${0.145/2} 0 ${0.875-0.029}" rpy="0 ${0/2} 0"/>
+  </joint>
+  <!-- ir_up_view -->
+  <link name="ir_up_view">
+    <collision>
+      <origin xyz="0 0 0" rpy="0 1.57 0"/>
+      <geometry>
+        <cylinder length="0.0004" radius="0.0001"/>
+      </geometry>
+    </collision>
+    <visual>
+      <origin xyz="0 0 0" rpy="0 1.57 0"/>
+      <geometry>
+        <cylinder length="0.0004" radius="0.0001"/>
+      </geometry>
+       <material name="Yellow">
+         <color rgba="1 1 0 1"/>
+       </material>
+    </visual>
+    <inertial>
+      <mass value="0.0"/>
+      <origin xyz="0 0 0" rpy="0 0 0"/>
+      <inertia ixx="1e-6" ixy="0" ixz="0" iyy="1e-6" iyz="0" izz="1e-6"/>
+    </inertial>
+  </link>
+  <gazebo reference="ir_up_view">
     <mu1 value="5.0"/>
     <mu2 value="5.0"/>
@@ -153,5 +189,5 @@
     <parent link="body_link"/>
     <child link="ir_down"/>
-    <origin xyz="${0.145/2} 0 ${0.275-0.029}" rpy="3.14 ${-1.57/2} 0"/>
+    <origin xyz="${0.145/2} 0 ${0.275-0.029}" rpy="0 -${ir_up_angle} 0"/>
     <axis xyz="0 0 1"/>
           <limit upper="1.57" lower="-1.57" velocity="50" effort="2"/>
@@ -193,4 +229,39 @@
   </link>
   <gazebo reference="ir_down">
+    <mu1 value="5.0"/>
+    <mu2 value="5.0"/>
+    <kp value="10000000.0"/>
+    <kd value="1.0"/>
+  </gazebo>
+  <!-- Body link /ir_down_view joint -->
+  <joint name="ir_down_view_joint" type="fixed">
+    <parent link="body_link"/>
+    <child link="ir_down_view"/>
+    <origin xyz="${0.145/2} 0 ${0.275-0.029}" rpy="0 0 0"/>
+  </joint>
+  <!-- ir_down_view -->
+  <link name="ir_down_view">
+    <collision>
+      <origin xyz="0 0 0" rpy="0 1.57 0"/>
+      <geometry>
+        <cylinder length="0.0004" radius="0.0001"/>
+      </geometry>
+    </collision>
+    <visual>
+      <origin xyz="0 0 0" rpy="0 1.57 0"/>
+      <geometry>
+        <cylinder length="0.0004" radius="0.0001"/>
+      </geometry>
+       <material name="Yellow">
+         <color rgba="1 1 0 1"/>
+       </material>
+    </visual>
+    <inertial>
+      <mass value="0.0"/>
+      <origin xyz="0 0 0" rpy="0 0 0"/>
+      <inertia ixx="1e-6" ixy="0" ixz="0" iyy="1e-6" iyz="0" izz="1e-6"/>
+    </inertial>
+  </link>
+  <gazebo reference="ir_down_view">
     <mu1 value="5.0"/>
     <mu2 value="5.0"/>

Commit message: add ir_tf_listener.cpp but stiil not work!

File: urdf/andbot.xacro (robot description, xacro)
@@ -6,5 +6,5 @@
   <xacro:property name="distance_between_wheels" value="0.3996"/>
   <xacro:property name="height_wheels_from_base" value="0.0392"/>
-  <xacro:property name="ir_up_angle" value="0.78539"/> <!--PI /4 -->
+  <xacro:property name="ir_up_angle" value="0"/> <!--PI /4 0.78539 -->
  <arg name="gui" value="true"/>
   <!-- Base footprint link-->
